File: Wiring Schematic/Project Titan/Hyperion.kicad_sch (KiCad schematic)
At the start: 0 parts

Commit message: Schematic Update
Parts:
- added A2: Motor Shield, PCM_arduino-library:Arduino_Uno_R2_Shield, symbol arduino-library:Arduino_Uno_R1_Shield
- added RF2: 433 mHz Receiver, symbol Connector_Generic_MountingPin:433_mHz_Receiver
- added U1: ATmega2560-16A, Package_QFP:TQFP-100_14x14mm_P0.5mm, symbol MCU_Microchip_ATmega:ATmega2560-16A
- added U5: IST8310, Package_LGA:LGA-16_3x3mm_P0.5mm, symbol Sensor_Magnetic:IST8310
- added U6 (x2): HC-SR04, HC-SR04:XCVR_HC-SR04, symbol HC-SR04:HC-SR04
Connections:
- new net: U5.11 (VSS), U5.9 (VSS)
- new net: U1.10 (VCC), U1.31 (VCC), U1.61 (VCC), U1.80 (VCC)
- new net: U1.11 (GND), U1.32 (GND), U1.62 (GND), U1.81 (GND), U1.99 (GND)
Other:
- note added: "Hyperion/Theia - Rover Board"
- note added: "Project Titan"
