File: Wiring Schematic/Project Titan/Project Titan.kicad_sch (KiCad schematic)
At the start: 9 parts, among them U1 ATmega2560-16A, U2 ATmega2560-16A, U3 HC-SR04, U4 NRF24L01, U5 NRF24L01, U6 HC-SR04, U7 HC-SR04, U8 LM2596S-ADJ

Commit message: Update
Parts:
- removed U4, U5: NRF24L01, Package_DFN_QFN:QFN-20-1EP_4x4mm_P0.5mm_EP2.5x2.5mm, symbol RF:NRF24L01
- added A2: Motor Shield, PCM_arduino-library:Arduino_Uno_R2_Shield, symbol arduino-library:Arduino_Uno_R1_Shield
- added D1: 3.5 TFT Display, symbol Display_Character:3.5_TFT
- added J1: 433 mHz Transmitter, symbol Connector_Generic_MountingPin:433_mHz_Transmitter
- added RF2: 433 mHz Receiver, symbol Connector_Generic_MountingPin:433_mHz_Receiver
- BT1: value Battery -> 5VDC
- U8: Schematic Name (none) -> Buck Boost
Connections:
- net at U2.9 (PE7): now also RF2.2 (Pin_2)
- net at BT1.1 (+): now also U8.1 (VIN)
- net at BT1.2 (-): now also U8.3 (GND)
Other:
- note added: "Hyperion/Theia - Rover Board"
- note added: "Schematic Notes: 5V DC and GND Net Labels are used for clarity."
- moved on the sheet: U1, U2

Commit message: Schematic Update
Other:
- added sheet Hyperion (Hyperion.kicad_sch)
Changed lines of the file:
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@@
+    )
+  )
+  (sheet (at -29.21 303.53) (size 478.79 293.37) (fields_autoplaced)
+    (stroke (width 0.1524) (type solid))
+    (fill (color 0 0 0 0.0000))
+    (property "Sheetname" "Hyperion" (at -29.21 300.9534 0)
+      (effects (font (size 5 5)) (justify left bottom))
+    )
+    (property "Sheetfile" "Hyperion.kicad_sch" (at -29.21 597.4846 0)
+      (effects (font (size 1.27 1.27)) (justify left top))
+    )
+    (instances
+      (project "Project Titan"
+        (path "/d057b949-c57e-49d7-8001-3a4b7593e964" (page "2"))
+      )
     )
   )

Commit message: Schematic Update
Parts:
- removed A2: Motor Shield, PCM_arduino-library:Arduino_Uno_R2_Shield, symbol arduino-library:Arduino_Uno_R1_Shield
- removed BT1: 5VDC, symbol Device:Battery
- removed D1: 3.5 TFT Display, symbol Display_Character:3.5_TFT
- removed J1: 433 mHz Transmitter, symbol Connector_Generic_MountingPin:433_mHz_Transmitter
- removed RF2: 433 mHz Receiver, symbol Connector_Generic_MountingPin:433_mHz_Receiver
- removed U1, U2: ATmega2560-16A, Package_QFP:TQFP-100_14x14mm_P0.5mm, symbol MCU_Microchip_ATmega:ATmega2560-16A
- removed U3, U6, U7: HC-SR04, HC-SR04:XCVR_HC-SR04, symbol HC-SR04:HC-SR04
- removed U8: LM2596S-ADJ, Package_TO_SOT_SMD:TO-263-5_TabPin3, symbol Regulator_Switching:LM2596S-ADJ
Other:
- added sheet RoverController (RoverController.kicad_sch)
- note added: "Notes: 5V DC and GND Net Labels are used for clarity."
- note added: "Project Titan"
- note removed: "Hyperion/Theia - Rover Board"
- note removed: "Schematic Notes: 5V DC and GND Net Labels are used for clarity."
- title: (none) -> Project Titan Block Diagram

Commit message: Schematic Update
Other:
- note added: "Arduino Mega"
- note removed: "Notes: 5V DC and GND Net Labels are used for clarity."
Changed lines of the file:
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@@
     (date "2025-04-22")
   )
+  (wire (pts (xy 293.37 185.42) (xy 327.66 185.42))
+    (stroke (width 1) (type default) (color 0 0 194 1))
+  )
+  (wire (pts (xy 241.3 199.39) (xy 241.3 209.55))
+    (stroke (width 1) (type default) (color 0 0 194 1))
+  )
   (wire (pts (xy 293.37 125.73) (xy 307.34 125.73))
+    (stroke (width 1) (type default) (color 0 0 194 1))
+  )
+  (wire (pts (xy 123.19 125.73) (xy 137.16 125.73))
     (stroke (width 1) (type default) (color 0 0 194 1))
   )
@@
     (stroke (width 1) (type default) (color 0 0 194 1))
   )
+  (wire (pts (xy 276.86 199.39) (xy 276.86 209.55))
+    (stroke (width 1) (type default) (color 0 0 194 1))
+  )
+  (wire (pts (xy 123.19 139.7) (xy 137.16 139.7))
+    (stroke (width 1) (type default) (color 0 0 194 1))
+  )
   (wire (pts (xy 78.74 104.14) (xy 78.74 88.9))
     (stroke (width 1) (type default) (color 255 0 0 1))
+  )
+  (wire (pts (xy 123.19 111.76) (xy 137.16 111.76))
+    (stroke (width 1) (type default) (color 0 0 194 1))
   )
   (wire (pts (xy 293.37 111.76) (xy 307.34 111.76))
     (stroke (width 1) (type default) (color 0 0 194 1))
   )
-  (wire (pts (xy 123.19 111.76) (xy 137.16 111.76))
+  (wire (pts (xy 327.66 165.1) (xy 327.66 185.42))
+    (stroke (width 1) (type default) (color 0 0 194 1))
+  )
+  (wire (pts (xy 123.19 153.67) (xy 137.16 153.67))
     (stroke (width 1) (type default) (color 0 0 194 1))
   )
@@
   )
   (text_box "433 MHz RF Transmitter"
+    (at 137.16 148.59 0) (size 67.31 10.16)
+    (stroke (width 1) (type default) (color 0 0 194 1))
+    (fill (type none))
+    (effects (font (size 3 3)))
+  )
+  (text_box "9V DC Battery"
+    (at 60.96 80.01 0) (size 38.1 8.89)
+    (stroke (width 1) (type default) (color 194 0 0 1))
+    (fill (type none))
+    (effects (font (size 3 3) (thickness 0.6) bold (color 0 0 0 1)))
+  )
+  (text_box "Debug Buttons"
     (at 137.16 106.68 0) (size 67.31 10.16)
     (stroke (width 1) (type default) (color 0 0 194 1))
@@
     (effects (font (size 3 3)))
   )
-  (text_box "9V DC"
-    (at 60.96 80.01 0) (size 38.1 8.89)
-    (stroke (width 1) (type default) (color 194 0 0 1))
+  (text_box "12V DC Motor"
+    (at 271.78 209.55 90) (size 10.16 39.37)
+    (stroke (width 1) (type default) (color 0 0 194 1))
     (fill (type none))
-    (effects (font (size 3 3) (thickness 0.6) bold (color 0 0 0 1)))
+    (effects (font (size 3 3)))
   )
   (text_box "QMC5883L Compass\n"
@@
     (stroke (width 1) (type default) (color 0 0 0 1))
     (fill (type none))
-    (effects (font (size 6 6)))
+    (effects (font (size 6 6) (thickness 1.2) bold))
+  )
+  (text_box "Mission Buttons"
+    (at 137.16 120.65 0) (size 67.31 10.16)
+    (stroke (width 1) (type default) (color 0 0 194 1))
+    (fill (type none))
+    (effects (font (size 3 3)))
   )
   (text_box "433 MHz RF Reciever"
@@
     (effects (font (size 3 3)))
   )
-  (text_box "5V DC/12V DC"
+  (text_box "12V DC Battery"
     (at 330.2 80.01 0) (size 43.18 8.89)
     (stroke (width 1) (type default) (color 194 0 0 1))
@@
     (stroke (width 1) (type default) (color 0 0 0 1))
     (fill (type none))
-    (effects (font (size 6 6)))
+    (effects (font (size 6 6) (thickness 1.2) bold))
   )
-  (text_box "Ultrasonic Distance Sensor"
+  (text_box "Ultrasonic Dist. Sensors"
     (at 226.06 106.68 0) (size 67.31 10.16)
     (stroke (width 1) (type default) (color 0 0 194 1))
@@
     (effects (font (size 3 3)))
   )
-  (text_box "Ultrasonic Distance Sensor"
+  (text_box "Adafruit REV 3 Motorshield"
+    (at 226.06 170.18 0) (size 67.31 29.21)
+    (stroke (width 1) (type default) (color 0 0 194 1))
+    (fill (type none))
+    (effects (font (size 3 3)))
+  )
+  (text_box "M100 GPS Module"
     (at 226.06 120.65 0) (size 67.31 10.16)
+    (stroke (width 1) (type default) (color 0 0 194 1))
+    (fill (type none))
+    (effects (font (size 3 3)))
+  )
+  (text_box "12V DC Motor"
+    (at 236.22 209.55 90) (size 10.16 39.37)
+    (stroke (width 1) (type default) (color 0 0 194 1))
+    (fill (type none))
+    (effects (font (size 3 3)))
+  )
+  (text_box "4.3\" TFT Display"
+    (at 137.16 134.62 0) (size 67.31 10.16)
     (stroke (width 1) (type default) (color 0 0 194 1))
     (fill (type none))
@@
     (effects (font (face "ROG Fonts") (size 7 7) (color 0 0 0 1)) (justify left bottom))
   )
-  (text "Notes: 5V DC and GND Net Labels are used for clarity."
-    (at 12.7 265.43 0)
-    (effects (font (size 1.27 1.27)) (justify left bottom))
+  (text "Arduino Mega" (at 325.12 147.32 0)
+    (effects (font (size 5 5)) (justify left bottom))
+  )
+  (text "Arduino Mega" (at 52.07 147.32 0)
+    (effects (font (size 5 5)) (justify left bottom))
   )
   (sheet (at -181.61 162.56) (size 123.19 110.49) (fields_autoplaced)
